Commit message: 小车通过ros_control控制了

File: src/bzzrobot_description/urdf/bzz2robot/actuator/wheel.urdf.xacro (robot description, xacro)
@@ -26,6 +26,6 @@
       <inertial>
         <origin xyz="0 0 0" rpy="0 0 0" />
-        <mass value="0.2" />
-        <inertia ixx="8.78e-5" ixy="0" ixz="0" iyy="8.78e-5" iyz="0" izz="2.05e-4" />
+        <mass value="0.5" />
+        <inertia ixx="0.001" ixy="0" ixz="0" iyy="0.001" iyz="0" izz="0.0005" />
       </inertial>
     </link>

File: src/bzzrobot_description/urdf/bzz2robot/base.urdf.xacro (robot description, xacro)
@@ -3,15 +3,4 @@
   <xacro:property name="base_radius" value="0.15" />
   <xacro:property name="base_length" value="0.20" />
-  <link name="base_footprint">
-    <visual>
-      <origin xyz="0 0 0" rpy="0 0 0" />
-      <geometry>
-        <sphere radius="0.01" />
-      </geometry>
-      <material name="base_footprint_material">
-        <color rgba="1.0 0.0 0.0 0.5" />
-      </material>
-    </visual>
-  </link>
   <link name="base_link">
     <!-- 基础链接可视化体 -->
@@ -39,4 +28,15 @@
       </inertial>
   </link>
+  <link name="base_footprint">
+    <visual>
+      <origin xyz="0 0 0" rpy="0 0 0" />
+      <geometry>
+        <sphere radius="0.01" />
+      </geometry>
+      <material name="base_footprint_material">
+        <color rgba="1.0 0.0 0.0 0.5" />
+      </material>
+    </visual>
+  </link>
   <joint name="base_footprint_joint" type="fixed">
     <parent link="base_footprint" />

File: src/bzzrobot_description/urdf/bzz2robot/bzz002.urdf.xacro (robot description, xacro)
@@ -9,12 +9,13 @@
   <xacro:include filename="$(find bzzrobot_description)/urdf/bzz2robot/actuator/wheel.urdf.xacro" />
   <xacro:include filename="$(find bzzrobot_description)/urdf/bzz2robot/actuator/caster.urdf.xacro" />
-  <xacro:include filename="$(find bzzrobot_description)/urdf/bzz2robot/plugins/gazebo_control_plugin.xacro" />
+  <!-- <xacro:include filename="$(find bzzrobot_description)/urdf/bzz2robot/plugins/gazebo_control_plugin.xacro" /> -->
   <xacro:include filename="$(find bzzrobot_description)/urdf/bzz2robot/plugins/gazebo_sensor_plugin.xacro" />
-  <!-- 相机光学坐标系link（虚拟部件） -->
+  <xacro:include filename="$(find bzzrobot_description)/urdf/bzz2robot/bzzbot.ros2_control.xacro" />
+  <!-- <xacro:include filename="$(find bzzrobot_description)/urdf/bzz2robot/plugins/gazebo_ros2_control.xacro" /> -->
   <link name="camera_link_optical" />
   <joint name="camera_joint_optical" type="fixed">
-      <parent link="camera_link" />
-      <child link="camera_link_optical" />
-      <origin xyz="0 0 0" rpy="0 ${pi/2} 0" />
+    <parent link="camera_link" />
+    <child link="camera_link_optical" />
+    <origin xyz="0 0 0" rpy="-1.5708 0 -1.5708" />
   </joint>
   <!-- 支持链接link -->
@@ -76,15 +77,15 @@
   <xacro:laser_plugin link_name="laser_link" />
   <xacro:imu_plugin link_name="imu_link" />
-  <xacro:depth_camera_plugin link_name="camera_link_optical" />
-  <!-- 两轮差速驱动插件 -->
+  <xacro:depth_camera_plugin link_name="camera_link" />
+ <!-- 两轮差速驱动插件
   <xacro:diff_drive_plugin
     left_joint="left_wheel_joint"
     right_joint="right_wheel_joint"
     wheel_separation="0.30"
-    wheel_radius="0.032" />
+    wheel_radius="0.032" /> -->
   <!-- 关节状态发布插件：将所有关节状态发布到 /joint_states -->
   <!-- 供 robot_state_publisher 使用以计算 TF 变换 -->
   <!-- 注意：caster关节是fixed类型，Gazebo中不存在continuous关节，所以只发布轮子关节 -->
-  <gazebo>
+  <!-- <gazebo>
     <plugin name="joint_state_publisher" filename="libgazebo_ros_joint_state_publisher.so">
       <joint_name>left_wheel_joint</joint_name>
@@ -92,4 +93,7 @@
       <publish_rate>50</publish_rate>
     </plugin>
-  </gazebo>
+  </gazebo> -->
+  <!-- ros2_control 插件 -->
+  <!-- 调用 bzzbot_ros2_control_plugin 宏，加载 ros2_control 硬件接口配置和 Gazebo 插件 -->
+  <xacro:bzzbot_ros2_control_plugin />
 </robot>

File: src/bzzrobot_description/urdf/bzz2robot/plugins/gazebo_sensor_plugin.xacro (robot description, xacro)
@@ -223,5 +223,5 @@
            - type="depth"：同时输出彩色图像和深度图像
       -->
-      <sensor name="camera_sensor" type="depth">
+      <sensor name="camera" type="depth">
         <!-- 传感器相对于link的位姿 -->
         <!-- 相机朝向由camera_link的joint origin控制，这里保持默认即可 -->
@@ -275,5 +275,5 @@
              plugin name="depth_camera" filename="libgazebo_ros_camera.so"：
              深度相机的Gazebo-ROS桥接插件
-             name="depth_camera"：插件实例名，必须唯一，节点名会是 /depth_camera_gazebo_ros
+             name="depth_cam  era"：插件实例名，必须唯一，节点名会是 /depth_camera_gazebo_ros
              filename="libgazebo_ros_camera.so"：同时支持普通相机和深度相机
              当sensor type="depth"时，自动发布深度相关话题
@@ -285,37 +285,15 @@
         <plugin name="depth_camera" filename="libgazebo_ros_camera.so">
           <ros>
-            <!-- namespace="/camera"：将所有相机话题放在 /camera 命名空间下 -->
-            <namespace>/camera</namespace>
+            <namespace>/</namespace>
+            <remapping>~/image_raw:=camera/image_raw</remapping>
+            <remapping>~/depth/image_raw:=camera/depth/image_raw</remapping>
+            <remapping>~/camera_info:=camera/camera_info</remapping>
+            <remapping>~/points:=camera/points</remapping>
           </ros>
-          <!--
-               frame_name="${link_name}"：数据的坐标系名称
-               这里是 camera_link，与相机所在的link一致
-          -->
-          <frame_name>${link_name}</frame_name>
-          <!--
-               hack_baseline：双目相机基线距离（米）
-               对于模拟深度相机，这个参数不影响实际测量，设为0.1即可
-          -->
+          <!-- 相机坐标系（默认是camera_link_optical）：发布深度图像和点云的坐标系 -->
+          <frame_name>camera_link_optical</frame_name>
           <hack_baseline>0.1</hack_baseline>
-          <!--
-               depth_camera：是否作为深度相机使用
-               true表示启用深度图像发布
-          -->
           <depth_camera>true</depth_camera>
-          <!--
-               image_topic：彩色图像话题名（在namespace下）
-               默认是 image_raw，所以完整话题是 /camera/image_raw
-          -->
-          <image_topic>image_raw</image_topic>
-          <!--
-               depth_image_topic：深度图像话题名（在namespace下）
-               默认是 depth/image_raw，完整话题是 /camera/depth/image_raw
-          -->
-          <depth_image_topic>depth/image_raw</depth_image_topic>
-          <!--
-               camera_info_topic：相机内参话题名（在namespace下）
-               默认是 camera_info，完整话题是 /camera/camera_info
-          -->
-          <camera_info_topic>camera_info</camera_info_topic>
+          <point_cloud>true</point_cloud>
         </plugin>
       </sensor>
